File: CAD/Ultimate_Co_Op_Mega_Shield/ultimate_Co-Op_v1_0.sch (EAGLE design)
At the start: 50 parts

Commit message: created a 'mini' version of the co-op board
Parts:
- ARDUINO_MEGA: device SparkFun-Boards:ARDUINO-MEGAFULL -> Nathans-Boards_small_mega:ARDUINO-MEGAFULL
Changed lines of the file:
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@@
 </classes>
 <parts>
-<part name="ARDUINO_MEGA" library="SparkFun-Boards" deviceset="ARDUINO-MEGA" device="FULL"/>
+<part name="ARDUINO_MEGA" library="Nathans-Boards_small_mega" deviceset="ARDUINO-MEGA" device="FULL"/>
 <part name="LED1" library="adafruit" deviceset="LED" device="5MM"/>
 <part name="R1" library="adafruit" deviceset="R-US_" device="0204/7" value="600"/>
