File: CAD/Ultimate_Co_Op_Mega_Shield/ultimate_Co-Op_v2_0.brd (EAGLE design)
At the start: 78.4 x 53.3 mm, 136 parts

Commit message: added updates to the ultimate co-op shield
Parts:
- added R11: 10k, adafruit:0204/7
- moved R10 27.3 mm to (17.8, 44.5), turned to 0 degrees
- moved POT 7.62 mm to (5.08, 20.3)
- moved R1 5.24 mm to (9.68, 11.7)
- moved R2 4.02 mm to (13.5, 11.7)
- moved R3 3.13 mm to (17.0, 11.7)
- moved LED3 2.84 mm to (20.5, 27.0)
- moved LED5 2.84 mm to (27.5, 27.0)
- moved LED1 2.84 mm to (13.5, 27.0)
- moved ROTARY 2.84 mm to (24.1, 39.4)
- moved LED7 2.84 mm to (34.4, 27.0)
- moved R9 2.54 mm to (36.8, 41.9)
- moved R4 2.29 mm to (20.5, 11.7)
- moved R8 2.29 mm to (34.4, 11.7)
- moved R7 1.69 mm to (31.1, 11.7)
- moved R5 1.50 mm to (24.1, 11.7)
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Connections:
- removed net POT1: ARDUINO_MEGA.A15, POT.2
- new net N$12: ARDUINO_MEGA.A15, R11.2
- new net N$15: POT.2, R11.1
Routing:
- net GND: track 15.2 -> 159.6 mm
- net OUT2_B: track 7.62 -> 108.4 mm, vias 0 -> 4
- net OUT1_START: track 7.62 -> 91.2 mm
- net ROTARY_3: track 0.00 -> 82.2 mm, vias 0 -> 1
- net ROTARY_2: track 0.00 -> 78.1 mm
- net ROTARY_1: track 0.00 -> 77.0 mm, vias 0 -> 2
- net OUT2_X: track 7.62 -> 77.9 mm, vias 0 -> 1
- net OUT1_DOWN: track 7.62 -> 76.2 mm
- net ROTARY_4: track 0.00 -> 67.8 mm, vias 0 -> 1
- net N$12: track 0.00 -> 66.0 mm
- net OUT2_A: track 7.62 -> 71.9 mm
- net OUT2_Y: track 7.62 -> 70.6 mm, vias 0 -> 1
- net 5V: track 0.00 -> 62.8 mm
- net OUT1_SELECT: track 7.62 -> 68.7 mm
- net OUT1_RIGHT: track 7.62 -> 67.9 mm, vias 0 -> 1
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Other:
- board text added: "1"
- board text added: "100"
- board text added: "2"
- board text added: "3"
- board text added: "4"
- board text added: "5"
- board text added: "6"
- board text added: "SNES Co-Op v2"
