File: CAD/Ultimate_Co_Op_Mega_Shield/ultimate_Co-Op_v2_0.sch (EAGLE design)
At the start: 136 parts

Commit message: added updates to the ultimate co-op shield
Parts:
- added R11: 10k, adafruit:R-US_0204/7
Connections:
- removed net POT1: ARDUINO_MEGA.A15(PK7), POT.2
- new net N$12: ARDUINO_MEGA.A15(PK7), R11.2
- new net N$15: POT.2, R11.1
Other:
- note added: "Ultimate SNES Co-Op Shield Revision 2.0 Designed by Nathan Villicana-Shaw Spring 2016"
- moved on the sheet: POT
Changed lines of the file:
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@@
 <layer number="91" name="Nets" color="2" fill="1" visible="yes" active="yes"/>
 <layer number="92" name="Busses" color="1" fill="1" visible="yes" active="yes"/>
-<layer number="93" name="Pins" color="2" fill="1" visible="no" active="yes"/>
+<layer number="93" name="Pins" color="2" fill="1" visible="yes" active="yes"/>
 <layer number="94" name="Symbols" color="4" fill="1" visible="yes" active="yes"/>
 <layer number="95" name="Names" color="7" fill="1" visible="yes" active="yes"/>
@@
 <part name="GND21" library="SparkFun-Aesthetics" deviceset="GND" device=""/>
 <part name="GND22" library="SparkFun-Aesthetics" deviceset="GND" device=""/>
+<part name="R11" library="adafruit" deviceset="R-US_" device="0204/7" value="10k"/>
 </parts>
 <sheets>
@@
 <text x="137.16" y="-30.48" size="3.81" layer="95">SNES OUTPUT #2</text>
 <frame x1="-91.44" y1="-162.56" x2="284.48" y2="114.3" columns="8" rows="5" layer="94"/>
+<text x="-76.2" y="-114.3" size="5.08" layer="94">Ultimate SNES Co-Op Shield
+            Revision 2.0
+           Designed by
+    Nathan Villicana-Shaw
+           Spring 2016</text>
 </plain>
 <instances>
@@
 <instance part="LED8" gate="G$1" x="53.34" y="-129.54" rot="R90"/>
 <instance part="R8" gate="G$1" x="43.18" y="-129.54"/>
-<instance part="GND9" gate="1" x="20.32" y="33.02" rot="R90"/>
+<instance part="GND9" gate="1" x="-45.72" y="33.02" rot="R90"/>
 <instance part="GND10" gate="1" x="109.22" y="-7.62" rot="R270"/>
 <instance part="GND11" gate="1" x="109.22" y="-132.08" rot="R270"/>
@@
 <instance part="GND12" gate="1" x="17.78" y="-10.16" rot="R270"/>
 <instance part="R9" gate="G$1" x="-22.86" y="88.9"/>
-<instance part="POT" gate="G$1" x="7.62" y="35.56"/>
+<instance part="POT" gate="G$1" x="-63.5" y="35.56"/>
 <instance part="IN_1" gate="G$1" x="-15.24" y="27.94"/>
 <instance part="IN_2" gate="G$1" x="-38.1" y="15.24"/>
@@
 <instance part="GND21" gate="1" x="-12.7" y="76.2" rot="R90"/>
 <instance part="GND22" gate="1" x="-12.7" y="88.9" rot="R90"/>
+<instance part="R11" gate="G$1" x="-33.02" y="38.1"/>
 </instances>
 <busses>
@@
 </segment>
 </net>
-<net name="POT1" class="0">
-<segment>
-<pinref part="ARDUINO_MEGA" gate="G$1" pin="A15(PK7)"/>
-<wire x1="27.94" y1="35.56" x2="15.24" y2="35.56" width="0.1524" layer="91"/>
-<pinref part="POT" gate="G$1" pin="2"/>
-</segment>
-</net>
 <net name="5V" class="0">
 <segment>
-<wire x1="15.24" y1="38.1" x2="20.32" y2="38.1" width="0.1524" layer="91"/>
-<label x="20.32" y="38.1" size="1.27" layer="95" xref="yes"/>
+<wire x1="-55.88" y1="38.1" x2="-45.72" y2="38.1" width="0.1524" layer="91"/>
+<label x="-45.72" y="38.1" size="1.27" layer="95" xref="yes"/>
 <pinref part="POT" gate="G$1" pin="3"/>
 </segment>
@@
 <pinref part="POT" gate="G$1" pin="1"/>
 <pinref part="GND9" gate="1" pin="GND"/>
-<wire x1="15.24" y1="33.02" x2="17.78" y2="33.02" width="0.1524" layer="91"/>
+<wire x1="-55.88" y1="33.02" x2="-48.26" y2="33.02" width="0.1524" layer="91"/>
 </segment>
 <segment>
@@
 <pinref part="ROTARY" gate="G$1" pin="7"/>
 <wire x1="-33.02" y1="73.66" x2="-30.48" y2="73.66" width="0.1524" layer="91"/>
+</segment>
+</net>
+<net name="N$12" class="0">
+<segment>
+<pinref part="ARDUINO_MEGA" gate="G$1" pin="A15(PK7)"/>
+<wire x1="27.94" y1="35.56" x2="-5.08" y2="35.56" width="0.1524" layer="91"/>
+<wire x1="-5.08" y1="35.56" x2="-7.62" y2="38.1" width="0.1524" layer="91"/>
+<wire x1="-7.62" y1="38.1" x2="-10.16" y2="38.1" width="0.1524" layer="91"/>
+<wire x1="-10.16" y1="38.1" x2="-12.7" y2="40.64" width="0.1524" layer="91"/>
+<wire x1="-12.7" y1="40.64" x2="-17.78" y2="40.64" width="0.1524" layer="91"/>
+<wire x1="-17.78" y1="40.64" x2="-20.32" y2="38.1" width="0.1524" layer="91"/>
+<pinref part="R11" gate="G$1" pin="2"/>
+<wire x1="-20.32" y1="38.1" x2="-27.94" y2="38.1" width="0.1524" layer="91"/>
+</segment>
+</net>
+<net name="N$15" class="0">
+<segment>
+<pinref part="R11" gate="G$1" pin="1"/>
+<wire x1="-38.1" y1="38.1" x2="-40.64" y2="35.56" width="0.1524" layer="91"/>
+<pinref part="POT" gate="G$1" pin="2"/>
+<wire x1="-40.64" y1="35.56" x2="-55.88" y2="35.56" width="0.1524" layer="91"/>
 </segment>
 </net>
@@
 </schematic>
 </drawing>
+<compatibility>
+<note version="6.3" minversion="6.2.2" severity="warning">
+Since Version 6.2.2 text objects can contain more than one line,
+which will not be processed correctly with this version.
+</note>
+</compatibility>
 </eagle>
